File: PCB/LibreServo_v1.brd (EAGLE design)
At the start: 44.5 x 39.5 mm, 66 parts

Commit message: LibreServo v1.c
Parts:
- removed C18, C7: 10uF, rcl:C0805
- removed R4, R5, R6: 160, rcl:R0402
- removed U$29, U$30: MICRO_PAD, Propio:MICRO_PAD
- added R_GREEN: 300, rcl:R0402
- added R_RED: 330, rcl:R0402
- C11, C12, C19, C20, C21, C8: value 10uF -> 22uF; device rcl:C0805 -> Propio:0805_MIN
- R1: device rcl:R1206 -> Propio:1206_ESTRECHA
- R12: value 160 -> 100
- R13: value 10K -> 100K
- R2: value 160 -> 1k1
- R_BLUE: value 160 -> 470
- U$27: device Propio:DPAK_SP -> Propio:SOT223_MOD
- moved R12 12.4 mm to (36.7, 31.9)
- moved R2 12.1 mm to (26.7, 32.4), turned to 180 degrees
- moved U$2 11.9 mm to (26.4, 29.9), turned to 180 degrees
- moved R11 11.8 mm to (39.1, 31.8), turned to 270 degrees
- moved C15 11.8 mm to (39.6, 28.2)
- moved U$10 10.9 mm to (37.6, 28.1)
- moved R1 10.6 mm to (27.7, 26.0), turned to 65 degrees
- moved R13 10.3 mm to (37.9, 32.4), turned to 270 degrees
- moved U$14 10.0 mm to (23.5, 34.0), flipped to the top, turned to 270 degrees
- moved U$13 10.0 mm to (41.6, 24.0), flipped to the top, turned to 90 degrees
- moved C21 9.42 mm to (27.9, 35.7), turned to 270 degrees
- moved C19 8.38 mm to (14.6, 8.59)
- moved C20 8.12 mm to (29.4, 35.7), turned to 270 degrees
- moved C14 7.63 mm to (26.3, 34.2), turned to 270 degrees
- moved C17 6.40 mm to (17.6, 7.37), turned to 270 degrees
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- renumbered R3 to R_BLUE
Connections:
- removed net N$4: U$1.7, U$29.P$1
- net +3V3_3: now also U$27.P$4; no longer C7.1, U$27.3
- net +7V_2_CABLE: now also C11.1, C12.1, C13.1, C14.1, C20.1, C21.1; no longer C11.2, C12.2, C13.2, C14.2, C20.2, C21.2
- net +7V_3: now also U$27.P$3; no longer C18.2, U$27.4
- net GND2: now also C11.2, C12.2, C13.2, C14.2, C20.2, C21.2; no longer C11.1, C12.1, C13.1, C14.1, C20.1, C21.1
- net GND3: now also U$27.P$1; no longer C18.1, C7.2, U$27.1
- net LED_GREEN: now also R_GREEN.2; no longer R4.2
- net LED_RED: now also R_RED.2; no longer R5.2
- net N$2: now also R_GREEN.1; no longer R4.1
- net N$3: now also R_RED.1; no longer R6.1
- net N$6: now also U$1.8; no longer R5.1, R6.2
- net N$7: now also U$1.7; no longer U$1.8, U$30.P$1
Routing:
- net EN_SERIAL_2: track 35.5 -> 9.89 mm
- net TX_2: track 8.27 -> 29.6 mm, vias 0 -> 1
- net TX_2_CABLE: track 40.0 -> 21.5 mm
- net RX_2: track 12.4 -> 25.9 mm, vias 0 -> 1
- net GND2: track 61.1 -> 68.3 mm, vias 2 -> 1
- net +7V_3: track 19.7 -> 12.8 mm
- net +7V_2_CABLE: track 31.5 -> 38.4 mm
- net +3V3_3: track 30.5 -> 23.6 mm, vias 2 -> 4
- net +7V_2: track 13.0 -> 19.4 mm
- net RX_2_CABLE: track 23.6 -> 17.3 mm, vias 0 -> 1
- net GND3: track 36.2 -> 30.6 mm
- net N$26: track 4.38 -> 8.46 mm
- net N$19: track 4.42 -> 8.37 mm
- net GND_1: track 69.9 -> 72.9 mm, vias 6 -> 7
- net V_CORRIENTE_2: track 16.2 -> 13.3 mm, vias 1 -> 0
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- added copper zone on layer 16, net +3V3_1
- added copper zone on layer 16, net +3V3_3
- added copper zone on layer 16, net +7V_1
- added copper zone on layer 16, net +7V_2
- added copper zone on layer 16, net +7V_2_CABLE
- added copper zone on layer 1, net GND2
- added copper zone on layer 1, net GND3
- added copper zone on layer 1, net GND_1
Other:
- board text added: "2x"
- board text added: "3V3"
- board text added: "3v3"
- board text added: "8MHz"
- board text added: "C1"
- board text added: "C10"
- board text added: "C16"
- board text added: "C17"
- board text added: "C8"
- board text added: "C9"
- board text added: "LibreServo v1.c"
- board text added: "R-B"
- board text added: "R-G"
- board text added: "R8"
- board text added: "R9"
- board text added: "RGB"
- board text added: "R_RED"
- board text added: "SN74LVC2"
- board text removed: "G"
- board text removed: "JST_PH-4"
- board text removed: "R"
- board text removed: "T"
