File: PCB/LibreServo_v1.sch (EAGLE design)
At the start: 66 parts

Commit message: LibreServo v1.c
Parts:
- removed C18, C7: 10uF, rcl:C-EUC0805
- removed R3, R4, R5, R6: 160, rcl:R-US_R0402
- removed U$29, U$30: MICRO_PAD, Propio:MICRO_PAD
- added R_BLUE: 470, rcl:R-US_R0402
- added R_GREEN: 300, rcl:R-US_R0402
- added R_RED: 330, rcl:R-US_R0402
- C11, C12, C19, C20, C21, C8: value 10uF -> 22uF; device rcl:C-EUC0805 -> Propio:C-EU0805-MIN
- R1: device rcl:R-US_R1206 -> Propio:R-US
- R12: value 160 -> 100
- R13: value 10K -> 100K
- R2: value 160 -> 1k1
- U$27: device Propio:NCP1117DT33G_SP -> Propio:NCP1117_MOD
Connections:
- removed net N$4: U$1.PA0, U$29.P$1
- net +3V3_3: now also U$27.P$4; no longer C7.1, U$27.P$2
- net +7V_2_CABLE: now also C11.1, C12.1, C13.1, C14.1, C20.1, C21.1; no longer C11.2, C12.2, C13.2, C14.2, C20.2, C21.2
- net +7V_3: no longer C18.2
- net GND2: now also C11.2, C12.2, C13.2, C14.2, C20.2, C21.2; no longer C11.1, C12.1, C13.1, C14.1, C20.1, C21.1
- net GND3: no longer C18.1, C7.2
- net LED_BLUE: now also R_BLUE.2; no longer R3.2
- net LED_GREEN: now also R_GREEN.2; no longer R4.2
- net LED_RED: now also R_RED.2; no longer R5.2
- net N$1: now also R_BLUE.1; no longer R3.1
- net N$2: now also R_GREEN.1; no longer R4.1
- net N$3: now also R_RED.1; no longer R6.1
- net N$6: now also U$1.PA1; no longer R5.1, R6.2
- net N$7: now also U$1.PA0; no longer U$1.PA1, U$30.P$1
Other:
- note added: "Alimentación"
- note added: "Bus entre PCBs"
- note added: "Comunicación Serie"
- note added: "Conectores"
- note added: "LED RGB"
- note added: "PCB 1"
- note added: "PCB 2"
- note added: "PCB 3"
- note added: "Potenciómetro"
- note added: "Puente en H"
- note added: "STM32F302K8"
- note added: "Sensor de Corriente"
- note added: "Sensor de Tensión"
- moved on the sheet: C1, C10, C11, C12, C13, C14, C15, C16, C17, C19, C2, C20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
